Commit message: Replace the single camera with a camera in each eye
The old camera sat between the eyes and, because camera_link was not
rotated with the body mesh, looked out of the fish's left side.

- mogi_bot.urdf: an eye_camera macro puts an invisible camera link in
  the centre of each robotic eye (positions from the eye properties),
  each looking out its own side 40 deg forward of sideways, like a
  real fish. Sides follow REP-103; the eye visual named
  right_robotic_eye is on the fish's left, so it holds left_eye_camera.
- mogi_bot.gazebo: one camera sensor per eye, same image, FOV, noise and
  water-hiding mask as before, publishing left_eye/ and right_eye/
  image and camera_info. 5 Hz each: two eyes at 10 Hz stalled the sim
  about once a second on integrated graphics (RTF 0.83 vs 0.99).
- Bridges, the color detector and the RViz camera displays now use the
  eye topics (the detector and RViz the left eye); READMEs updated.

File: src/fishy_fish_navigation/urdf/mogi_bot.urdf (robot description, URDF)
Before this commit: robot mogi_bot, 11 links, 10 joints
Links:
- removed link camera_link
- removed link camera_link_optical
Joints:
- removed joint camera_joint
- removed joint camera_optical_joint
